Commit message: add lula motion planning (rmpflow); implement first simple action-sequence carried out on needle-transfer task

File: data/dVRK/PSM/psm_col.urdf (robot description, URDF)
Before this commit: robot psm_col_updated_joint, 14 links, 13 joints
Links:
- link psm_main_insertion_link: geometry 
- link psm_main_insertion_link_2: geometry 
- link psm_main_insertion_link_3: geometry 
- link psm_pitch_end_link: geometry 
- link psm_remote_center_link: geometry 
- link psm_tool_gripper1_link: geometry 
- link psm_tool_gripper2_link: geometry 
- link psm_tool_pitch_link: geometry 
- link psm_tool_roll_link: geometry 
- link psm_tool_yaw_link: geometry 
Joints:
- joint psm_main_insertion_joint: limit lower=0.0565 upper=0.24 effort=6000. velocity=0. -> lower=0.0565 upper=0.24 effort=12.0 velocity=1.0
- joint psm_pitch_end_joint: limit lower=-0.9251 upper=0.9251 effort=6000. velocity=2.0999999 -> lower=-0.9251 upper=0.9251 effort=12.0 velocity=1.0
- joint psm_tool_gripper1_joint: limit lower=-0.5235988 upper=0. effort=1200. velocity=2.0999999 -> lower=-0.5235988 upper=0. effort=0.1 velocity=0.2
- joint psm_tool_gripper2_joint: limit lower=0. upper=0.5235988 effort=1200. velocity=2.0999999 -> lower=0. upper=0.5235988 effort=0.1 velocity=0.2
- joint psm_tool_pitch_joint: limit lower=-1.3962999 upper=1.3962999 effort=6000. velocity=2.0999999 -> lower=-1.3962999 upper=1.3962999 effort=12.0 velocity=1.0
- joint psm_tool_roll_joint: limit lower=-4.5378997 upper=4.5378997 effort=6000. velocity=2.0999999 -> lower=-4.5378997 upper=4.5378997 effort=12.0 velocity=1.0
- joint psm_tool_yaw_joint: limit lower=-0.5235988 upper=0.5235988 effort=6000. velocity=2.0999999 -> lower=-0.5235988 upper=0.5235988 effort=12.0 velocity=1.0
- joint psm_yaw_joint: limit lower=-1.5883 upper=1.5883 effort=6000. velocity=2.0999999 -> lower=-1.5883 upper=1.5883 effort=12.0 velocity=1.0
